File: storm32bgc v120 rev2/STorM32 BGC v1202.brd (EAGLE design)
At the start: 50 x 50 mm, 93 parts, among them IC1 STM32F103RCT6, IC10 TC4452DFN08, IC11 TC4452DFN08, IC12 74AHC1G86DBV, IC13 MPU6050, IC14 BT HC06, IC2 NCP1117ST33T3G, IC3 TC4452DFN08, IC4 TC4452DFN08, IC5 TC4452DFN08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

Commit message: v1.2 rev2
Parts:
- R11: value 2.2k -> 1.5k
Changed lines of the file:
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@@
 <grid distance="0.003125" unitdist="inch" unit="inch" style="lines" multiple="1" display="yes" altdistance="0.025" altunitdist="inch" altunit="inch"/>
 <layers>
-<layer number="1" name="Top" color="4" fill="1" visible="no" active="yes"/>
+<layer number="1" name="Top" color="4" fill="1" visible="yes" active="yes"/>
 <layer number="2" name="Route2" color="1" fill="3" visible="no" active="no"/>
 <layer number="3" name="Route3" color="4" fill="3" visible="no" active="no"/>
@@
 <layer number="14" name="Route14" color="1" fill="6" visible="no" active="no"/>
 <layer number="15" name="Route15" color="4" fill="6" visible="no" active="no"/>
-<layer number="16" name="Bottom" color="1" fill="1" visible="yes" active="yes"/>
+<layer number="16" name="Bottom" color="1" fill="1" visible="no" active="yes"/>
 <layer number="17" name="Pads" color="2" fill="1" visible="yes" active="yes"/>
 <layer number="18" name="Vias" color="2" fill="1" visible="yes" active="yes"/>
 <layer number="19" name="Unrouted" color="6" fill="1" visible="yes" active="yes"/>
 <layer number="20" name="Dimension" color="15" fill="1" visible="yes" active="yes"/>
-<layer number="21" name="tPlace" color="7" fill="1" visible="no" active="yes"/>
-<layer number="22" name="bPlace" color="7" fill="1" visible="yes" active="yes"/>
-<layer number="23" name="tOrigins" color="15" fill="1" visible="no" active="yes"/>
-<layer number="24" name="bOrigins" color="15" fill="1" visible="yes" active="yes"/>
-<layer number="25" name="tNames" color="7" fill="1" visible="no" active="yes"/>
-<layer number="26" name="bNames" color="7" fill="1" visible="yes" active="yes"/>
-<layer number="27" name="tValues" color="7" fill="1" visible="no" active="yes"/>
+<layer number="21" name="tPlace" color="7" fill="1" visible="yes" active="yes"/>
+<layer number="22" name="bPlace" color="7" fill="1" visible="no" active="yes"/>
+<layer number="23" name="tOrigins" color="15" fill="1" visible="yes" active="yes"/>
+<layer number="24" name="bOrigins" color="15" fill="1" visible="no" active="yes"/>
+<layer number="25" name="tNames" color="7" fill="1" visible="yes" active="yes"/>
+<layer number="26" name="bNames" color="7" fill="1" visible="no" active="yes"/>
+<layer number="27" name="tValues" color="7" fill="1" visible="yes" active="yes"/>
 <layer number="28" name="bValues" color="7" fill="1" visible="no" active="yes"/>
 <layer number="29" name="tStop" color="7" fill="3" visible="no" active="yes"/>
@@
 <layer number="37" name="tTest" color="7" fill="1" visible="no" active="yes"/>
 <layer number="38" name="bTest" color="7" fill="1" visible="no" active="yes"/>
-<layer number="39" name="tKeepout" color="4" fill="11" visible="no" active="yes"/>
-<layer number="40" name="bKeepout" color="1" fill="11" visible="yes" active="yes"/>
-<layer number="41" name="tRestrict" color="4" fill="10" visible="no" active="yes"/>
-<layer number="42" name="bRestrict" color="1" fill="10" visible="yes" active="yes"/>
+<layer number="39" name="tKeepout" color="4" fill="11" visible="yes" active="yes"/>
+<layer number="40" name="bKeepout" color="1" fill="11" visible="no" active="yes"/>
+<layer number="41" name="tRestrict" color="4" fill="10" visible="yes" active="yes"/>
+<layer number="42" name="bRestrict" color="1" fill="10" visible="no" active="yes"/>
 <layer number="43" name="vRestrict" color="2" fill="10" visible="yes" active="yes"/>
 <layer number="44" name="Drills" color="7" fill="1" visible="no" active="yes"/>
@@
 <layer number="49" name="Reference" color="7" fill="1" visible="yes" active="yes"/>
 <layer number="50" name="dxf" color="7" fill="1" visible="no" active="no"/>
-<layer number="51" name="tDocu" color="7" fill="1" visible="no" active="yes"/>
-<layer number="52" name="bDocu" color="7" fill="1" visible="yes" active="yes"/>
+<layer number="51" name="tDocu" color="7" fill="1" visible="yes" active="yes"/>
+<layer number="52" name="bDocu" color="7" fill="1" visible="no" active="yes"/>
 <layer number="53" name="tGND_GNDA" color="7" fill="9" visible="no" active="no"/>
 <layer number="54" name="bGND_GNDA" color="1" fill="9" visible="no" active="no"/>
@@
 <wire x1="8.493125" y1="41.275" x2="8.493125" y2="38.57625" width="0.1016" layer="25"/>
 <wire x1="8.493125" y1="41.275" x2="8.651875" y2="41.275" width="0.1016" layer="25"/>
+<rectangle x1="12.7" y1="41.036875" x2="14.9225" y2="45.005625" layer="31"/>
+<rectangle x1="12.7" y1="35.321875" x2="14.9225" y2="39.290625" layer="31"/>
+<rectangle x1="12.7" y1="29.606875" x2="14.9225" y2="33.575625" layer="31"/>
+<rectangle x1="26.67" y1="41.036875" x2="28.8925" y2="45.005625" layer="31"/>
+<rectangle x1="26.67" y1="35.321875" x2="28.8925" y2="39.290625" layer="31"/>
+<rectangle x1="26.67" y1="29.606875" x2="28.8925" y2="33.575625" layer="31"/>
+<rectangle x1="40.9575" y1="29.606875" x2="43.18" y2="33.575625" layer="31"/>
+<rectangle x1="40.9575" y1="35.321875" x2="43.18" y2="39.290625" layer="31"/>
+<rectangle x1="40.9575" y1="41.036875" x2="43.18" y2="45.005625" layer="31"/>
 </plain>
 <attributes>
@@
 <attribute name="VALUE" x="12.28725" y="6.778625" size="0.8128" layer="27"/>
 </element>
-<element name="R11" library="rcl" package="R0603" value="2.2k" x="10.95375" y="9.525" smashed="yes" rot="R180">
+<element name="R11" library="rcl" package="R0603" value="1.5k" x="10.95375" y="9.525" smashed="yes" rot="R180">
 <attribute name="VALUE" x="12.98575" y="8.397875" size="0.7112" layer="27" rot="R90"/>
 </element>
@@
 <contactref element="JP8" pad="1"/>
 <contactref element="C13" pad="-"/>
-<polygon width="0.1524" layer="1" isolate="0.000203125" rank="6">
+<polygon width="0.1524" layer="1" isolate="0.1524" rank="6">
 <vertex x="0" y="0"/>
 <vertex x="0" y="50"/>
@@
 <vertex x="50" y="0"/>
 </polygon>
-<polygon width="0.1524" layer="16" isolate="0.000203125" rank="6">
+<polygon width="0.1524" layer="16" isolate="0.1524" rank="6">
 <vertex x="0" y="0"/>
 <vertex x="0" y="50"/>
