File: storm32bgc v120 rev2/STorM32 BGC v1202.sch (EAGLE design)
At the start: 93 parts, among them IC1 STM32F103RCT6, IC10 TC4452DFN08, IC11 TC4452DFN08, IC12 74AHC1G86DBV, IC13 MPU6050, IC14 BT HC06, IC2 NCP1117ST33T3G, IC3 TC4452DFN08, IC4 TC4452DFN08, IC5 TC4452DFN08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

Commit message: v1.2 rev2
Other:
- note added: "11. Mar. 2014"
- note added: "Schaltplan v1.2 rev2"
- note removed: "9. Feb. 2014"
- note removed: "Schaltplan v1.2 rev1"
Changed lines of the file:
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@@
 <sheet>
 <plain>
-<text x="180.34" y="-38.1" size="2.54" layer="91">9. Feb. 2014</text>
+<text x="180.34" y="-38.1" size="2.54" layer="91">11. Mar. 2014</text>
 <text x="180.34" y="-43.18" size="2.54" layer="91">(c) www.olliw.eu</text>
 <text x="180.34" y="-27.94" size="2.54" layer="91">STorM32-BGC</text>
-<text x="180.34" y="-33.02" size="2.54" layer="91">Schaltplan v1.2  rev1</text>
+<text x="180.34" y="-33.02" size="2.54" layer="91">Schaltplan v1.2  rev2</text>
 <text x="178.435" y="-23.495" size="1.778" layer="97">This is a open source hardware project, under the terms
 of the TAPR Open Hardware License, http://www.tapr.org/ohl.html.
@@
 XOR:  PC4
 (unused ports: PA4,PC5,PC12,PD2)</text>
-<text x="180.34" y="-220.98" size="2.54" layer="91">9. Feb. 2014</text>
+<text x="180.34" y="-220.98" size="2.54" layer="91">11. Mar. 2014</text>
 <text x="180.34" y="-226.06" size="2.54" layer="91">(c) www.olliw.eu</text>
 <text x="180.34" y="-210.82" size="2.54" layer="91">STorM32-BGC</text>
-<text x="180.34" y="-215.9" size="2.54" layer="91">Schaltplan v1.2  rev1</text>
+<text x="180.34" y="-215.9" size="2.54" layer="91">Schaltplan v1.2  rev2</text>
 <text x="178.435" y="-206.375" size="1.778" layer="97">This is a open source hardware project, under the terms
 of the TAPR Open Hardware License, http://www.tapr.org/ohl.html.
@@
 - all parts named/valued properly to produce good BOM
 rev1
-- value of R11 changed to 1.5k</text>
+- value of R11 changed to 1.5k
+rev2
+- DFN packages cream added
+- DFN packages silk a bit improved</text>
 <text x="137.16" y="12.7" size="1.778" layer="95">JP1</text>
 <text x="259.08" y="6.35" size="1.778" layer="95">JP2</text>
