File: storm32-nt-modules/storm32-nt-motor-module-v009-eagle-gerber-files-20150630/STorM32 NT motor module v009.brd (EAGLE design)
At the start: 39.4 x 19.7 mm, 34 parts, among them IC1 NCP1117ST50T3G, U1 STM32F10XTXU6, Y1 RESONATORSMD

Commit message: nt motor module initial release
Parts:
- SJ3: value ID1 -> ID2
- SJ4: value ID2 -> ID1
- moved SJ3 0.16 mm to (20.0, 14.9)
Other:
- board text added: "NT motor module v0.09"
- board text added: "NTB IN"
- board text added: "P - - R X - Y - X"
- board text removed: "M0 - - M1 X - M2 - X"
- board text removed: "NT motor module v0.08"
- board text removed: "NTB-IN"
Changed lines of the file:
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@@
 <text x="4.7625" y="1.666875" size="1.27" layer="25" font="vector" ratio="15" rot="R180">IN</text>
 <text x="21.11375" y="19.05" size="1.6764" layer="26" font="vector" ratio="15" rot="MR180">www.olliw.eu</text>
-<text x="32.22625" y="5.3975" size="1.27" layer="26" font="vector" ratio="15" rot="MR180">VBAT</text>
-<text x="29.21" y="5.3975" size="1.27" layer="26" font="vector" ratio="15" rot="MR180">5V</text>
-<text x="0.3175" y="10.00125" size="1.016" layer="26" font="vector" ratio="15" rot="MR180">VBAT</text>
-<text x="0.9525" y="1.42875" size="1.016" layer="26" font="vector" ratio="15" rot="MR180">GND</text>
-<text x="26.51125" y="2.2225" size="1.016" layer="26" font="vector" ratio="15" rot="MR180">GND</text>
-<text x="25.55875" y="9.68375" size="1.016" layer="26" font="vector" ratio="15" rot="MR180">VBAT</text>
+<text x="32.385" y="5.3975" size="1.27" layer="26" font="vector" ratio="15" rot="MR180">VBAT</text>
+<text x="29.05125" y="5.3975" size="1.27" layer="26" font="vector" ratio="15" rot="MR180">5V</text>
+<text x="0.3175" y="10.00125" size="1.016" layer="26" font="vector" ratio="20" rot="MR180">VBAT</text>
+<text x="0.9525" y="1.42875" size="1.016" layer="26" font="vector" ratio="20" rot="MR180">GND</text>
+<text x="26.51125" y="2.2225" size="1.016" layer="26" font="vector" ratio="20" rot="MR180">GND</text>
+<text x="25.55875" y="9.68375" size="1.016" layer="26" font="vector" ratio="20" rot="MR180">VBAT</text>
 <text x="6.985" y="19.05" size="1.6764" layer="26" font="vector" ratio="15" rot="MR180" align="bottom-center">NT motor
 module
-v0.08</text>
+v0.09</text>
 <text x="31.27375" y="5.318125" size="1.016" layer="25" font="vector" ratio="15">Tx</text>
 <text x="31.27375" y="3.889375" size="1.016" layer="25" font="vector" ratio="15">Rx</text>
@@
 <rectangle x1="26.19375" y1="7.62" x2="28.41625" y2="11.43" layer="31"/>
 <rectangle x1="26.19375" y1="1.905" x2="28.41625" y2="5.715" layer="31"/>
-<text x="10.95375" y="1.74625" size="1.27" layer="26" font="vector" ratio="15" rot="MR180">LED1</text>
-<text x="20.79625" y="0.47625" size="1.27" layer="26" font="vector" ratio="15" rot="MR0">LED2</text>
-<text x="8.41375" y="7.62" size="1.27" layer="26" font="vector" ratio="15" rot="MR270">NTB-IN</text>
-<text x="38.735" y="8.89" size="1.27" layer="26" font="vector" ratio="15" rot="SMR270">NTB-OUT</text>
+<text x="14.76375" y="0.635" size="1.016" layer="26" font="vector" ratio="20" rot="MR0">LED1</text>
+<text x="19.05" y="0.635" size="1.016" layer="26" font="vector" ratio="20" rot="MR0">LED2</text>
+<text x="6.35" y="6.35" size="1.27" layer="26" font="vector" ratio="15" rot="MR180" align="bottom-center">NTB
+IN</text>
+<text x="38.735" y="8.5725" size="1.27" layer="26" font="vector" ratio="15" rot="SMR270">NTB-OUT</text>
 <text x="38.735" y="15.24" size="1.27" layer="26" font="vector" ratio="15" rot="SMR270">MOT</text>
-<text x="19.52625" y="14.12875" size="1.016" layer="26" font="vector" ratio="15" rot="MR180">M0 - -
-M1 X -
-M2 - X</text>
+<text x="19.05" y="14.12875" size="1.27" layer="26" font="vector" ratio="20" rot="MR180">P - -
+R X -
+Y - X</text>
 </plain>
 <attributes>
@@
 <attribute name="VALUE" x="32.2849" y="6.82625" size="0.02" layer="28" rot="MR180"/>
 </element>
-<element name="SJ3" library="# SparkFun2" package="SJ_2S-NO" value="ID1" x="20.16125" y="14.9225" smashed="yes" rot="MR90">
-<attribute name="VALUE" x="18.51025" y="14.0145" size="0.4064" layer="28" rot="MR90"/>
-</element>
-<element name="SJ4" library="# SparkFun2" package="SJ_2S-NO" value="ID2" x="21.9075" y="14.9225" smashed="yes" rot="MR90">
+<element name="SJ3" library="# SparkFun2" package="SJ_2S-NO" value="ID2" x="20.0025" y="14.9225" smashed="yes" rot="MR90">
+<attribute name="VALUE" x="18.3515" y="14.0145" size="0.4064" layer="28" rot="MR90"/>
+</element>
+<element name="SJ4" library="# SparkFun2" package="SJ_2S-NO" value="ID1" x="21.9075" y="14.9225" smashed="yes" rot="MR90">
 <attribute name="VALUE" x="20.2565" y="14.0145" size="0.4064" layer="28" rot="MR90"/>
 </element>
@@
 <via x="13.335" y="8.255" extent="1-16" drill="0.3048"/>
 <via x="15.08125" y="2.38125" extent="1-16" drill="0.4"/>
-<via x="38.1" y="12.3825" extent="1-16" drill="0.4"/>
-<via x="38.1" y="14.9225" extent="1-16" drill="0.4"/>
+<via x="38.1" y="11.58875" extent="1-16" drill="0.4"/>
+<via x="38.1" y="15.71625" extent="1-16" drill="0.4"/>
 <via x="38.1" y="17.4625" extent="1-16" drill="0.4"/>
 <via x="38.1" y="9.8425" extent="1-16" drill="0.4"/>
@@
 <wire x1="11.5325" y1="16.6125" x2="12.3825" y2="16.6125" width="0.4064" layer="1"/>
 <wire x1="12.1675" y1="9.36625" x2="11.1125" y2="9.36625" width="0.4064" layer="1"/>
-<via x="15.001875" y="16.8275" extent="1-16" drill="0.3048"/>
-<wire x1="15.001875" y1="16.8275" x2="16.906875" y2="16.8275" width="0.3048" layer="16"/>
+<via x="14.843125" y="16.8275" extent="1-16" drill="0.3048"/>
+<wire x1="14.843125" y1="16.8275" x2="16.906875" y2="16.8275" width="0.3048" layer="16"/>
 <wire x1="16.906875" y1="16.8275" x2="17.541875" y2="17.4625" width="0.3048" layer="16"/>
 <wire x1="17.541875" y1="17.4625" x2="19.05" y2="17.4625" width="0.3048" layer="16"/>
@@
 <via x="20.716875" y="16.589375" extent="1-16" drill="0.3048"/>
 <wire x1="19.05" y1="18.415" x2="19.05" y2="17.4625" width="0.3048" layer="16"/>
-<wire x1="15.001875" y1="16.8275" x2="14.605" y2="16.8275" width="0.3048" layer="1"/>
+<wire x1="14.843125" y1="16.8275" x2="14.605" y2="16.8275" width="0.3048" layer="1"/>
 <wire x1="14.605" y1="16.8275" x2="14.0890625" y2="16.3909375" width="0.3048" layer="1"/>
 <wire x1="12.3825" y1="10.810875" x2="11.20775" y2="10.810875" width="0.1524" layer="1"/>
@@
 <wire x1="21.3675" y1="10.85875" x2="21.510625" y2="10.715625" width="0.1524" layer="1"/>
 <via x="21.510625" y="10.715625" extent="1-16" drill="0.3048"/>
-<wire x1="21.510625" y1="10.715625" x2="20.16125" y2="12.065" width="0.1524" layer="16"/>
-<wire x1="20.16125" y1="12.065" x2="20.16125" y2="14.5415" width="0.1524" layer="16"/>
+<wire x1="21.510625" y1="10.715625" x2="20.0025" y2="12.22375" width="0.1524" layer="16"/>
+<wire x1="20.0025" y1="12.22375" x2="20.0025" y2="14.5415" width="0.1524" layer="16"/>
 </signal>
 <signal name="N$4">
