File: storm32-nt/storm32-nt-bgc-v330m/STorM32 NT BGC v330m.brd (EAGLE design)
At the start: 25 x 40 mm, 74 parts, among them IC1 STM32F103RCT6, IC2 MPU9250, IC3 LMR14206, IC4 TC1185-3.3VCT713, IC5 CP2102N-QFN20, IC6 TJA1051TK/3, IC7 74AHC1G86, Q1 RESSMD

Commit message: v33m BOM improved
Parts:
- Q1: value RESSMD -> 8MHz
Changed lines of the file:
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@@
 </element>
 <element name="D1" library="# stdlib" package="SOD123W-DIODE" value="PMEG3010ER" x="20.79625" y="7.3025" smashed="yes" rot="R90"/>
-<element name="Q1" library="# SparkFun2" package="RESONATOR-SMD" value="RESSMD" x="28.2575" y="22.225" smashed="yes" rot="R270"/>
+<element name="Q1" library="# SparkFun2" package="RESONATOR-SMD" value="8MHz" x="28.2575" y="22.225" smashed="yes" rot="R270"/>
 <element name="RESET" library="# stdlib" package="TACTILE-SWITCH-SMD-RIGHT-TL1014" value="R" x="15.39875" y="1.984375" smashed="yes"/>
 <element name="USB" library="# SparkFun2" package="USB-MICROB" value="Amphenol 10118192-0001LF" x="7.3025" y="10.715625" smashed="yes" rot="R270"/>
