File: storm32-nt/storm32-nt-bgc-v330m/STorM32 NT BGC v330m.sch (EAGLE design)
At the start: 74 parts, among them IC1 STM32F103RCT6, IC2 MPU9250, IC3 LMR14206, IC4 TC1185-3.3VCT713, IC5 CP2102N-QFN20, IC6 TJA1051TK/3, IC7 74AHC1G86, Q1 RESSMD

Commit message: v33m BOM improved
Parts:
- Q1: value RESSMD -> 8MHz
Changed lines of the file:
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@@
 <part name="GND34" library="# supply1" deviceset="GND" device=""/>
 <part name="D1" library="# stdlib" deviceset="DIODE-SCHOTTKY" device="SOD123-W" value="PMEG3010ER"/>
-<part name="Q1" library="# SparkFun2" deviceset="RESONATOR" device="SMD" value="RESSMD"/>
+<part name="Q1" library="# SparkFun2" deviceset="RESONATOR" device="SMD" value="8MHz"/>
 <part name="RESET" library="# stdlib" deviceset="SWITCH-SMD-RIGHT-TL1014" device="" value="R"/>
 <part name="USB" library="# SparkFun2" deviceset="USB" device="-MICROB" value="Amphenol 10118192-0001LF"/>
