File: storm32-nt/storm32-nt-motor-v42EC-g4/T STorM32 NT motor v42ECg4 001.brd (EAGLE design)
At the start: 29 x 29 mm, 37 parts, among them IC1 STM32G431KBUx, IC2 LDO-TLV767, IC3 TLE5012B E1000X, IC9 DRV8311, Q1 CSTCE8M00G55-R0

Commit message: update of STorM32 NT Motor module v4.2EC G4, few corrections&updates (thx to qvertigo)
Parts:
- Q1: value CSTCE8M00G55-R0 -> CSTNE8M00GH5C000R0
Changed lines of the file:
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@@
 <attribute name="VALUE" x="14.605" y="5.23875" size="0.8128" layer="28" rot="MR0"/>
 </element>
-<element name="Q1" library="# SparkFun2" package="RESONATOR-SMD" value="CSTCE8M00G55-R0" x="19.685" y="5.55625" smashed="yes" rot="R90"/>
+<element name="Q1" library="# SparkFun2" package="RESONATOR-SMD" value="CSTNE8M00GH5C000R0" x="19.685" y="5.55625" smashed="yes" rot="R90"/>
 <element name="LED1" library="led" package="CHIPLED_0603" value="red" x="11.27125" y="15.875" smashed="yes" rot="R180">
 <attribute name="VALUE" x="13.81125" y="16.98625" size="0.8128" layer="27" rot="R180"/>
