File: storm32-nt/storm32-nt-motor-v42EC-g4/T STorM32 NT motor v42ECg4 001.sch (EAGLE design)
At the start: 37 parts, among them IC1 STM32G431KBUx, IC2 LDO-TLV767, IC3 TLE5012B E1000X, IC9 DRV8311, Q1 CSTCE8M00G55-R0

Commit message: update of STorM32 NT Motor module v4.2EC G4, few corrections&updates (thx to qvertigo)
Parts:
- Q1: value CSTCE8M00G55-R0 -> CSTNE8M00GH5C000R0
Other:
- note added: "001: - update of ceramic Q1 to newer - correct pin labels - add comment on curr sense support"
- note added: "GAIN may have to be wired according to your need"
- note added: "Note: curr sense is not yet supported Modules which do not want to support curr sense should wire PA1,PA2, PA3 to ground (this will allow firmware to detect this). Derived schemes may then be simplified, e.g., not include the RC filters and the related wiring."
- note added: "PA9 Tx PA10 Rx PA8 PHASE1 (T1_CH1) PA11 PHASE2 (T1_CH4, T4_CH1) PA12 PHASE3 (T4_CH2, T16_CH1) PB5 LED PB6 ID1 PB7 ID2 PA5 SCK PA6 MISO PA7 MOSI PB0 CS PA1 CURRENT3 PA2 CURRENT2 PA3 CURRENT1"
- note added: "curr sense is not yet supported -> in DIY builds these RC filters do not need to be populated"
- note removed: "PA9 Tx PA10 Rx PA8 PHASE1 (T1_CH1) PA11 PHASE2 (T1_CH4, T4_CH1) PA12 PHASE3 (T4_CH2, T16_CH1) PB5 LED PB6 ID1 PB7 ID2 PA5 SCK PA6 MISO PA7 MOSI PB0 CS PA1 CURRENT1 PA2 CURRENT2 PA3 CURRENT3"
- note removed: "curr sense is not yet supported -> these RC filters do not need to be populated -> derived schemes may be simplified and not include/wire them"
Changed lines of the file:
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@@
 <part name="GND6" library="# supply1" deviceset="GND" device=""/>
 <part name="GND8" library="# supply1" deviceset="GND" device=""/>
-<part name="Q1" library="# SparkFun2" deviceset="RESONATOR" device="SMD" value="CSTCE8M00G55-R0"/>
+<part name="Q1" library="# SparkFun2" deviceset="RESONATOR" device="SMD" value="CSTNE8M00GH5C000R0"/>
 <part name="LED1" library="led" deviceset="LED" device="CHIPLED_0603" value="red"/>
 <part name="GND12" library="# supply1" deviceset="GND" device=""/>
@@
 PA7   MOSI
 PB0   CS
-PA1   CURRENT1
+PA1   CURRENT3
 PA2   CURRENT2
-PA3   CURRENT3</text>
+PA3   CURRENT1</text>
 <text x="129.54" y="55.88" size="1.778" layer="91" align="top-left">INLA, INLB, INLC = AVDD (or to wire for global disable)
 MODE = highZ: 3x mode, 9A OCP, AVDD: 3x mode, 5A OCP
@@
 convenience</text>
 <text x="226.06" y="7.62" size="1.778" layer="91" align="top-left">curr sense is not yet supported
--&gt; these RC filters do not need
-to be populated
--&gt; derived schemes may be
-simplified and not include/wire
-them</text>
+-&gt; in DIY builds these RC filters
+do not need to be populated</text>
+<text x="285.115" y="65.405" size="1.778" layer="97" align="top-left">001:
+- update of ceramic Q1 to newer
+- correct pin labels
+- add comment on curr sense support</text>
+<text x="129.54" y="40.64" size="1.778" layer="91" align="top-left">GAIN may have to be wired according to your need</text>
+<text x="284.48" y="50.8" size="1.778" layer="91" align="top-left">Note: curr sense is not yet supported
+Modules which do not want to
+support curr sense should wire PA1,PA2,
+PA3 to ground (this will allow firmware to
+detect this).
+Derived schemes may then be simplified,
+e.g., not include the RC filters and the
+related wiring.</text>
 </plain>
 <instances>
